File: TinyTX4.sch (EAGLE design)
At the start: 47 parts, among them IC1 ATTINY84, IC2 IC2

Commit message: Layoutkorrektur - retry
Gehäuse für LT3525 auf SC70 geändert. (2. Versuch)
Changed lines of the file:
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@@
 <?xml version="1.0" encoding="utf-8"?>
 <!DOCTYPE eagle SYSTEM "eagle.dtd">
-<eagle version="6.4">
+<eagle version="6.5.0">
 <drawing>
 <settings>
